Commit message: added methods in the IK class Changed filename paths to the URDF file

File: robot_movement/URDF/dofbot.urdf (robot description, URDF)
Before this commit: robot dofbot, 6 links, 5 joints
Links:
- link base_link: geometry collision mesh filename=file://meshes/base_link.STL; visual mesh filename=file://meshes/base_link.STL
- link link1: geometry collision mesh filename=file://meshes/link1.STL; visual mesh filename=file://meshes/link1.STL
- link link2: geometry collision mesh filename=file://meshes/link2.STL; visual mesh filename=file://meshes/link2.STL
- link link3: geometry collision mesh filename=file://meshes/link3.STL; visual mesh filename=file://meshes/link3.STL
- link link4: geometry collision mesh filename=file://meshes/link4.STL; visual mesh filename=file://meshes/link4.STL
- link link5: geometry collision mesh filename=file://meshes/link5.STL; visual mesh filename=file://meshes/link5.STL

Commit message: Add files via upload

File: robot_movement/URDF/dofbot.urdf (robot description, URDF)
Before this commit: robot dofbot, 6 links, 5 joints
Links:
- link base_link: geometry collision mesh filename=package://dofbot_moveit/meshes/base_link.STL; visual mesh filename=package://dofbot_moveit/meshes/base_link.STL
- link link1: geometry collision mesh filename=package://dofbot_moveit/meshes/link1.STL; visual mesh filename=package://dofbot_moveit/meshes/link1.STL
- link link2: geometry collision mesh filename=package://dofbot_moveit/meshes/link2.STL; visual mesh filename=package://dofbot_moveit/meshes/link2.STL
- link link3: geometry collision mesh filename=package://dofbot_moveit/meshes/link3.STL; visual mesh filename=package://dofbot_moveit/meshes/link3.STL
- link link4: geometry collision mesh filename=package://dofbot_moveit/meshes/link4.STL; visual mesh filename=package://dofbot_moveit/meshes/link4.STL
- link link5: geometry collision mesh filename=package://dofbot_moveit/meshes/link5.STL; visual mesh filename=package://dofbot_moveit/meshes/link5.STL
Joints:
- joint joint5: origin xyz=-0.07385 -0.001 0 rpy=0 -1.57 0 -> xyz=-0.17385 -0.001 0 rpy=0 -1.57 0
